File: I2CRJ45X16.sch (EAGLE design)
At the start: 51 parts, among them IC1 MCP23017SO, IC2 MCP23017SO, J1 M06-SOCKET, J2 M06-SOCKET, J3 M02X3-PIN, J4 M02X3-PIN

Commit message: Routing
Parts:
- removed J4: M02X3-PIN, SuperHouse-Connectors:M02X3-PIN
- removed U$1: RJ45-X8, SuperHouse-Connectors:RJ45-X8
- added C3, C4: 10uF, SuperHouse-DiscreteSemi:CAP0805
- added C7: 330uF, SuperHouse-DiscreteSemi:CAP_POLG
- added IC3, IC4: MCP23017SO, SuperHouse-ICs:MCP23017SO
- added R41, R42, R43, R44, R45, R46, R47, R48, R49, R50, R51, R52, R53, R54, R55, R56, R57, R58, R59, R60, R61, R62, R63, R64, R65, R66: 1K, SuperHouse-DiscreteSemi:RESISTOR0603
- added R67, R68, R69: 10K, SuperHouse-DiscreteSemi:RESISTOR0603
- added SJ1: I2C Address, SuperHouse-Jumpers:SJ-NORMAL
- added SJ2: SCL PU, SuperHouse-Jumpers:SJ-NORMAL
- added SJ3: SDA PU, SuperHouse-Jumpers:SJ-NORMAL
- J1, J2: value M06-SOCKET -> RJ45-X8; device SuperHouse-Connectors:M06-SOCKET -> SuperHouse-Connectors:RJ45-X8
- J3: value M02X3-PIN -> M06-SOCKET; device SuperHouse-Connectors:M02X3-PIN -> SuperHouse-Connectors:M06-SOCKET
- R33, R34, R35, R36, R37, R38: value 10K -> 1K
- R39, R40: value 10K -> 2K2
Connections:
- net GPA0 renamed GPA0-1
- net GPA1 renamed GPA1-1
- net GPA2 renamed GPA2-1
- net GPA3 renamed GPA3-1
- net GPA4 renamed GPA4-1
- net GPA5 renamed GPA5-1
- net GPA6 renamed GPA6-1
- net GPA7 renamed GPA7-1
- net GPB0 renamed GPB0-1
- net GPB1 renamed GPB1-1
- net GPB2 renamed GPB2-1
- net GPB3 renamed GPB3-1
- net GPB4 renamed GPB4-1
- net GPB5 renamed GPB5-1
- net GPB6 renamed GPB6-1
- net GPB7 renamed GPB7-1
- removed net A1: R1.2, U$1.A1
- removed net A2: R3.2, U$1.A2
- removed net A3: R2.2, U$1.A3
- removed net A6: R4.2, U$1.A6
- removed net B1: R15.2, U$1.B1
- removed net B2: R13.2, U$1.B2
- removed net B3: R11.2, U$1.B3
- removed net B6: R9.2, U$1.B6
- removed net C1: R17.2, U$1.C1
- removed net C2: R19.2, U$1.C2
- removed net C3: R18.2, U$1.C3
- removed net C6: R20.2, U$1.C6
- removed net D1: R31.2, U$1.D1
- removed net D2: R29.2, U$1.D2
- removed net D3: R27.2, U$1.D3
- removed net D6: R25.2, U$1.D6
- removed net E1: R7.2, U$1.E1
- removed net E2: R6.2, U$1.E2
- removed net E3: R5.2, U$1.E3
- removed net E6: R8.2, U$1.E6
- removed net F1: R16.2, U$1.F1
- removed net F2: R14.2, U$1.F2
- removed net F3: R12.2, U$1.F3
- removed net F6: R10.2, U$1.F6
- removed net G1: R23.2, U$1.G1
- removed net G2: R22.2, U$1.G2
- removed net G3: R21.2, U$1.G3
- removed net G6: R24.2, U$1.G6
- removed net H1: R32.2, U$1.H1
- removed net H2: R30.2, U$1.H2
- removed net H3: R28.2, U$1.H3
- removed net H6: R26.2, U$1.H6
- removed net N$3: IC1.A1, J3.3, R34.2
- removed net N$4: IC1.A0, J3.1, R33.2
- removed net N$5: IC2.A0, J4.1, R36.2
- removed net N$6: IC2.A2, J4.5, R38.2
- new net 1A1: J1.A1, R1.2
- new net 1A2: J1.A2, R3.2
- new net 1A3: J1.A3, R2.2
- new net 1A6: J1.A6, R4.2
- new net 1B1: J1.B1, R15.2
- new net 1B2: J1.B2, R13.2
- new net 1B3: J1.B3, R11.2
- new net 1B6: J1.B6, R9.2
- new net 1C1: J1.C1, R17.2
- new net 1C2: J1.C2, R19.2
- new net 1C3: J1.C3, R18.2
- new net 1C6: J1.C6, R20.2
- new net 1D1: J1.D1, R31.2
- new net 1D2: J1.D2, R29.2
- new net 1D3: J1.D3, R27.2
- new net 1D6: J1.D6, R25.2
- new net 1E1: J1.E1, R7.2
- new net 1E2: J1.E2, R6.2
- new net 1E3: J1.E3, R5.2
- new net 1E6: J1.E6, R8.2
- new net 1F1: J1.F1, R16.2
- new net 1F2: J1.F2, R14.2
- new net 1F3: J1.F3, R12.2
- new net 1F6: J1.F6, R10.2
- new net 1G1: J1.G1, R23.2
- new net 1G2: J1.G2, R22.2
- new net 1G3: J1.G3, R21.2
- new net 1G6: J1.G6, R24.2
- new net 1H1: J1.H1, R32.2
- new net 1H2: J1.H2, R30.2
- new net 1H3: J1.H3, R28.2
- new net 1H6: J1.H6, R26.2
- new net 2A1: J2.A1, R33.2
- new net 2A2: J2.A2, R35.2
- new net 2A3: J2.A3, R34.2
- new net 2A6: J2.A6, R36.2
- new net 2B1: J2.B1, R49.2
- new net 2B2: J2.B2, R47.2
- new net 2B3: J2.B3, R45.2
- new net 2B6: J2.B6, R43.2
- new net 2C1: J2.C1, R51.2
- new net 2C2: J2.C2, R53.2
- new net 2C3: J2.C3, R52.2
- new net 2C6: J2.C6, R54.2
- new net 2D1: J2.D1, R65.2
- new net 2D2: J2.D2, R63.2
- new net 2D3: J2.D3, R61.2
- new net 2D6: J2.D6, R59.2
- new net 2E1: J2.E1, R41.2
- new net 2E2: J2.E2, R38.2
- new net 2E3: J2.E3, R37.2
- new net 2E6: J2.E6, R42.2
- new net 2F1: J2.F1, R50.2
- new net 2F2: J2.F2, R48.2
- new net 2F3: J2.F3, R46.2
- new net 2F6: J2.F6, R44.2
- new net 2G1: J2.G1, R57.2
- new net 2G2: J2.G2, R56.2
- new net 2G3: J2.G3, R55.2
- new net 2G6: J2.G6, R58.2
- new net 2H1: J2.H1, R66.2
- new net 2H2: J2.H2, R64.2
- new net 2H3: J2.H3, R62.2
- new net 2H6: J2.H6, R60.2
- new net ADDR2: IC1.A2, IC2.A2, IC3.A2, IC4.A2, R67.2, SJ1.1
- new net GPA0-3: IC3.GPA0, R33.1
- new net GPA0-4: IC4.GPA0, R51.1
- new net GPA1-3: IC3.GPA1, R35.1
- new net GPA1-4: IC4.GPA1, R53.1
- new net GPA2-3: IC3.GPA2, R34.1
- new net GPA2-4: IC4.GPA2, R52.1
- new net GPA3-3: IC3.GPA3, R36.1
- new net GPA3-4: IC4.GPA3, R54.1
- new net GPA4-3: IC3.GPA4, R41.1
- new net GPA4-4: IC4.GPA4, R57.1
- new net GPA5-3: IC3.GPA5, R38.1
- new net GPA5-4: IC4.GPA5, R56.1
- new net GPA6-3: IC3.GPA6, R37.1
- new net GPA6-4: IC4.GPA6, R55.1
- new net GPA7-3: IC3.GPA7, R42.1
- new net GPA7-4: IC4.GPA7, R58.1
- new net GPB0-3: IC3.GPB0, R49.1
- new net GPB0-4: IC4.GPB0, R65.1
- new net GPB1-3: IC3.GPB1, R47.1
- new net GPB1-4: IC4.GPB1, R63.1
- new net GPB2-3: IC3.GPB2, R45.1
- new net GPB2-4: IC4.GPB2, R61.1
- new net GPB3-3: IC3.GPB3, R43.1
- new net GPB3-4: IC4.GPB3, R59.1
- new net GPB4-3: IC3.GPB4, R50.1
- new net GPB4-4: IC4.GPB4, R66.1
- new net GPB5-3: IC3.GPB5, R48.1
- new net GPB5-4: IC4.GPB5, R64.1
- new net GPB6-3: IC3.GPB6, R46.1
- new net GPB6-4: IC4.GPB6, R62.1
- new net GPB7-3: IC3.GPB7, R44.1
- new net GPB7-4: IC4.GPB7, R60.1
- net !INT: now also IC3.INTA, IC4.INTA, J3.6; no longer J1.6, J2.6
- net GND: now also C3.2, C4.2, C7.-, IC1.A0, IC1.A1, IC2.A1, IC3.A0, IC3.VSS, IC4.VSS, J1.A7, J1.A8, J1.B7, J1.B8, J1.C7, J1.C8, J1.D7, J1.D8, J1.E7, J1.E8, J1.F7, J1.F8, J1.G7, J1.G8, J1.GND0, J1.GND1, J1.GND2, J1.GND3, J1.GND4, J1.GND5, J1.H7, J1.H8, J2.A7, J2.A8, J2.B7, J2.B8, J2.C7, J2.C8, J2.D7, J2.D8, J2.E7, J2.E8, J2.F7, J2.F8, J2.G7, J2.G8, J2.GND0, J2.GND1, J2.GND2, J2.GND3, J2.GND4, J2.GND5, J2.H7, J2.H8, J3.4, R67.1; no longer J1.4, J2.4, R33.1, R34.1, R35.1, R36.1, R37.1, R38.1, U$1.A7, U$1.A8, U$1.B7, U$1.B8, U$1.C7, U$1.C8, U$1.D7, U$1.D8, U$1.E7, U$1.E8, U$1.F7, U$1.F8, U$1.G7, U$1.G8, U$1.H7, U$1.H8
- net N$1: now also R68.2, SJ2.1; no longer IC2.A1, J4.3, R37.2
- net N$2: now also R69.2, SJ3.1; no longer IC1.A2, J3.5, R35.2
- net SCL: now also IC3.SCL, IC4.SCL, J3.2, R68.1; no longer J1.2, J2.2
- net SDA: now also IC3.SDA, IC4.SDA, J3.1, R69.1; no longer J1.1, J2.1
- net VCC: now also C3.1, C4.1, IC2.A0, IC3.!RESET, IC3.A1, IC3.VDD, IC4.!RESET, IC4.A0, IC4.A1, IC4.VDD, J3.3, SJ1.2, SJ2.2, SJ3.2; no longer J1.3, J2.3, J3.2, J3.4, J3.6, J4.2, J4.4, J4.6
- net VIN: now also C7.+, J1.A4, J1.A5, J1.B4, J1.B5, J1.C4, J1.C5, J1.D4, J1.D5, J1.E4, J1.E5, J1.F4, J1.F5, J1.G4, J1.G5, J1.H4, J1.H5, J2.A4, J2.A5, J2.B4, J2.B5, J2.C4, J2.C5, J2.D4, J2.D5, J2.E4, J2.E5, J2.F4, J2.F5, J2.G4, J2.G5, J2.H4, J2.H5, J3.5; no longer J1.5, J2.5, U$1.A4, U$1.A5, U$1.B4, U$1.B5, U$1.C4, U$1.C5, U$1.D4, U$1.D5, U$1.E4, U$1.E5, U$1.F4, U$1.F5, U$1.G4, U$1.G5, U$1.H4, U$1.H5
Other:
- note added: "I2C Addr: 0x20/0x24"
- note added: "I2C Addr: 0x21/0x25"
- note added: "I2C Addr: 0x22/0x26"
- note added: "I2C Addr: 0x23/0x27"
- note added: "I2C to 16 x RJ45 Breakout"
- note added: "SKU: I2C16RJ45"
- note added: "V1.0 (2019-08-15)"
- note added: "www.superhouse.tv/i2c16rj45"
- note removed: "GND VCC VIN SDA SCL interrupts?"
- note removed: "I2C to RJ45 Breakout"
- note removed: "SKU: I2CRJ45"
- note removed: "V1.0 (2019-07-25)"
- note removed: "www.superhouse.tv/i2crj45"
