File: I2C16RJ45.brd (EAGLE design)
At the start: 146 x 50 mm, 86 parts, among them IC1 MCP23017SO, IC2 MCP23017SO, IC3 MCP23017SO, IC4 MCP23017SO, J1 RJ45-X8, J2 RJ45-X8, J3 M06-SOCKET

Commit message: Board and schematic labelling
Other:
- board text added: "16 Channel I2C RJ45 Breakout"
- board text added: "SKU: I2CRJ45X16"
- board text added: "VIN: 12V"
- board text added: "www.superhouse.tv/i2crj45x16"
- board text removed: "I2C to 16xRJ45 Breakout"
- board text removed: "SKU: I2C16RJ45"
- board text removed: "VIN: 5-24V"
- board text removed: "www.superhouse.tv/i2c16rj45"
Changed lines of the file:
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@@
 <?xml version="1.0" encoding="utf-8"?>
 <!DOCTYPE eagle SYSTEM "eagle.dtd">
-<eagle version="9.4.2">
+<eagle version="9.5.0">
 <drawing>
 <settings>
@@
 <layer number="19" name="Unrouted" color="12" fill="1" visible="yes" active="yes"/>
 <layer number="20" name="Dimension" color="15" fill="1" visible="yes" active="yes"/>
-<layer number="21" name="tPlace" color="15" fill="1" visible="no" active="yes"/>
-<layer number="22" name="bPlace" color="14" fill="1" visible="no" active="yes"/>
+<layer number="21" name="tPlace" color="15" fill="1" visible="yes" active="yes"/>
+<layer number="22" name="bPlace" color="14" fill="1" visible="yes" active="yes"/>
 <layer number="23" name="tOrigins" color="15" fill="1" visible="yes" active="yes"/>
 <layer number="24" name="bOrigins" color="15" fill="1" visible="yes" active="yes"/>
@@
 </layers>
 <board>
-<fusionsync huburn="a.cGVyc29uYWw6dWUyZDliZmNi" projecturn="a.cGVyc29uYWw6dWUyZDliZmNiIzIwMTkwNjE5MTk5NjgzNjgx" f3durn="urn:adsk.wipprod:dm.lineage:_H2PRmvNSomCkomNSTRBxw" pcbguid="e014f554-0983-42e7-88b6-f6e08b18e2c7" lastpulledtime="" lastsyncedchangeguid="e428ff5b-e486-0e1a-3b0f-55ed86d9a8bf"/>
+<fusionsync huburn="a.cGVyc29uYWw6dWUyZDliZmNi" projecturn="a.cGVyc29uYWw6dWUyZDliZmNiIzIwMTkwNjE5MTk5NjgzNjgx" f3durn="urn:adsk.wipprod:dm.lineage:_H2PRmvNSomCkomNSTRBxw" pcbguid="e014f554-0983-42e7-88b6-f6e08b18e2c7" lastpulledtime="" lastsyncedchangeguid="306704fd-182e-ea57-2995-b1876d038e4d"/>
 <plain>
 <wire x1="3" y1="0" x2="0" y2="3" width="0" layer="20" curve="-90"/>
@@
 <wire x1="143" y1="0" x2="3" y2="0" width="0" layer="20"/>
 <text x="138.953" y="7.623" size="1.4224" layer="21" font="vector" ratio="17">v1.0</text>
-<text x="37.455" y="47.354" size="1.6764" layer="21" font="vector" ratio="17" align="bottom-center">www.superhouse.tv/i2c16rj45</text>
-<text x="31.191" y="45.171" size="1.27" layer="21" font="vector" ratio="17">SKU: I2C16RJ45</text>
+<text x="37.455" y="47.354" size="1.6764" layer="21" font="vector" ratio="17" align="bottom-center">www.superhouse.tv/i2crj45x16</text>
+<text x="31.191" y="45.171" size="1.27" layer="21" font="vector" ratio="17">SKU: I2CRJ45X16</text>
 <hole x="3" y="3" drill="3.2"/>
 <hole x="143" y="3" drill="3.2"/>
@@
 <text x="73.455" y="28.854" size="2.54" layer="21" font="vector" ratio="17" distance="30" align="bottom-center">Super
 House</text>
-<text x="77.955" y="47.354" size="2" layer="21" font="vector" ratio="17" distance="30">I2C to 16xRJ45 Breakout</text>
+<text x="76.955" y="47.354" size="1.8" layer="21" font="vector" ratio="17" distance="30">16 Channel I2C RJ45 Breakout</text>
 <text x="101.955" y="45.354" size="1.6764" layer="21" font="vector" ratio="17" distance="30">by Jon Oxer</text>
 <text x="131.455" y="31.854" size="1.6764" layer="22" font="vector" ratio="17" distance="30" rot="MR0">Copyright 2019 SuperHouse Automation Pty Ltd
@@
 <circle x="3" y="3" radius="3.201559375" width="0.254" layer="42"/>
 <text x="2.877" y="7.953" size="1.4224" layer="21" font="vector" ratio="17" rot="R90">VCC: 1.8-5.5V</text>
-<text x="4.877" y="7.953" size="1.4224" layer="21" font="vector" ratio="17" rot="R90">VIN: 5-24V</text>
+<text x="4.877" y="7.953" size="1.4224" layer="21" font="vector" ratio="17" rot="R90">VIN: 12V</text>
 <text x="62" y="28.5" size="1.4224" layer="22" font="vector" ratio="18" rot="MR0">1: Data 1
 2: Data 2

Commit message: Added fiducials
Parts:
- added FID1, FID2, FID3: FIDUCIAL1X2.5, freetronics:FIDUCIAL-1X2.5
